Commit message: Cập nhật package assem_urdf

File: urdf/assem_urdf.urdf.xacro (robot description, xacro)
@@ -96,5 +96,5 @@
     type="continuous">
     <origin
-      xyz="-0.036511 -0.099997 0.0198"
+      xyz="-0.036511 -0.098 0.0198"
       rpy="1.5708 0 0" />
     <parent
@@ -152,5 +152,5 @@
     type="continuous">
     <origin
-      xyz="-0.036511 0.099997 0.0198"
+      xyz="-0.036511 0.098 0.0198"
       rpy="-1.5708 0 0" />
     <parent
@@ -312,6 +312,6 @@
     <joint name="wheel_right_joint">
       <command_interface name="velocity">
-        <param name="min">-1</param>
-        <param name="max">1</param>
+        <param name="min">-3.1416</param>
+        <param name="max">3.1416</param>
       </command_interface>
       <state_interface name="position"/>
@@ -321,6 +321,6 @@
     <joint name="wheel_left_joint">
       <command_interface name="velocity">
-        <param name="min">-1</param>
-        <param name="max">1</param>
+        <param name="min">-3.1416</param>
+        <param name="max">3.1416</param>
       </command_interface>
       <state_interface name="position"/>
@@ -330,7 +330,23 @@
   </ros2_control>
   <gazebo>
+    <!-- Plugin gz_ros2_control-system -->
+    <!-- Đây là plugin kết nối Gazebo với ROS 2 Control, cho phép điều khiển robot trong môi trường mô phỏng -->
+    <!-- Plugin này tạo giao diện giữa các joint trong mô phỏng và hệ thống điều khiển ROS 2 -->
     <plugin filename="ign_ros2_control-system" name="ign_ros2_control::IgnitionROS2ControlPlugin">
       <parameters>$(find assem_urdf)/config/control.yaml</parameters>
     </plugin>
+    <!-- Collision properties -->
+    <collision>
+      <!-- max_contacts: Số lượng điểm tiếp xúc tối đa cho phép khi có va chạm -->
+      <max_contacts>20</max_contacts>
+      <contact>
+        <ode>
+          <!-- max_vel: Vận tốc tối đa cho phép khi có va chạm (100.0 m/s) -->
+          <max_vel>100.0</max_vel>
+          <!-- min_depth: Độ sâu tối thiểu để xem là có va chạm (0.001m = 1mm) -->
+          <min_depth>0.001</min_depth>
+        </ode>
+      </contact>
+    </collision>
   </gazebo>
 </robot>

Commit message: Update assem_urdf package

File: urdf/assem_urdf.urdf.xacro (robot description, xacro)
@@ -273,4 +273,39 @@
       xyz="0 0 0" />
   </joint>
+  <gazebo reference="lidar_link">
+    <sensor name="lidar_sensor" type="gpu_lidar">
+      <pose>0 0 0 0 0 0</pose>
+      <ignition_frame_id>lidar_link</ignition_frame_id>
+      <topic>/scan</topic>
+      <update_rate>10</update_rate>
+      <ray>
+        <scan>
+          <horizontal>
+            <samples>360</samples>
+            <resolution>1</resolution>
+            <min_angle>-3.14159265</min_angle>
+            <max_angle>3.14159265</max_angle>
+          </horizontal>
+          <vertical>
+            <samples>1</samples>
+            <resolution>1</resolution>
+            <min_angle>0</min_angle>
+            <max_angle>0</max_angle>
+          </vertical>
+        </scan>
+        <range>
+          <min>0.15</min>
+          <max>12.0</max>
+          <resolution>0.01</resolution>
+        </range>
+      </ray>
+      <noise>
+        <type>gaussian</type>
+        <mean>0.0</mean>
+        <stddev>0.01</stddev>
+      </noise>
+      <visualize>true</visualize>
+    </sensor>
+  </gazebo>
   <!-- ============================================= -->
   <!-- Caster - Stabilization wheel                 -->
@@ -312,6 +347,6 @@
     <joint name="wheel_right_joint">
       <command_interface name="velocity">
-        <param name="min">-3.1416</param>
-        <param name="max">3.1416</param>
+        <param name="min">-31.416</param>
+        <param name="max">31.416</param>
       </command_interface>
       <state_interface name="position"/>
@@ -321,6 +356,6 @@
     <joint name="wheel_left_joint">
       <command_interface name="velocity">
-        <param name="min">-3.1416</param>
-        <param name="max">3.1416</param>
+        <param name="min">-31.416</param>
+        <param name="max">31.416</param>
       </command_interface>
       <state_interface name="position"/>
@@ -330,19 +365,12 @@
   </ros2_control>
   <gazebo>
-    <!-- Plugin gz_ros2_control-system -->
-    <!-- Đây là plugin kết nối Gazebo với ROS 2 Control, cho phép điều khiển robot trong môi trường mô phỏng -->
-    <!-- Plugin này tạo giao diện giữa các joint trong mô phỏng và hệ thống điều khiển ROS 2 -->
     <plugin filename="ign_ros2_control-system" name="ign_ros2_control::IgnitionROS2ControlPlugin">
       <parameters>$(find assem_urdf)/config/control.yaml</parameters>
     </plugin>
-    <!-- Collision properties -->
-    <collision>
-      <!-- max_contacts: Số lượng điểm tiếp xúc tối đa cho phép khi có va chạm -->
+    <collision>
       <max_contacts>20</max_contacts>
       <contact>
         <ode>
-          <!-- max_vel: Vận tốc tối đa cho phép khi có va chạm (100.0 m/s) -->
           <max_vel>100.0</max_vel>
-          <!-- min_depth: Độ sâu tối thiểu để xem là có va chạm (0.001m = 1mm) -->
           <min_depth>0.001</min_depth>
         </ode>
@@ -350,3 +378,42 @@
     </collision>
   </gazebo>
+  <gazebo reference="camera_link">
+    <sensor type="depth" name="depth_camera">
+      <update_rate>30.0</update_rate>
+      <camera name="depth_camera">
+        <pose>0 0 0 0 0 0</pose>
+        <horizontal_fov>1.3962634</horizontal_fov>
+        <image>
+          <width>640</width>
+          <height>480</height>
+          <format>R8G8B8</format>
+        </image>
+        <clip>
+          <near>0.005</near>
+          <far>10.0</far>
+        </clip>
+      </camera>
+      <cameraName>depth_camera</cameraName>
+      <alwaysOn>true</alwaysOn>
+      <updateRate>10</updateRate>
+      <imageTopicName>rgb/image_raw</imageTopicName>
+      <depthImageTopicName>depth/image_raw</depthImageTopicName>
+      <pointCloudTopicName>depth/points</pointCloudTopicName>
+      <cameraInfoTopicName>rgb/camera_info</cameraInfoTopicName>
+      <depthImageCameraInfoTopicName>depth/camera_info</depthImageCameraInfoTopicName>
+      <gz_frame_id>camera_link</gz_frame_id>
+      <pointCloudCutoff>0.5</pointCloudCutoff>
+      <pointCloudCutoffMax>3.0</pointCloudCutoffMax>
+      <hackBaseline>0.07</hackBaseline>
+      <distortionK1>0.0</distortionK1>
+      <distortionK2>0.0</distortionK2>
+      <distortionK3>0.0</distortionK3>
+      <distortionT1>0.0</distortionT1>
+      <distortionT2>0.0</distortionT2>
+      <CxPrime>0</CxPrime>
+      <Cx>0</Cx>
+      <Cy>0</Cy>
+      <focalLength>0</focalLength>
+    </sensor>
+  </gazebo>
 </robot>

Commit message: Update assem_urdf package with latest changes

File: urdf/assem_urdf.urdf.xacro (robot description, xacro)
@@ -277,5 +277,5 @@
       <pose>0 0 0 0 0 0</pose>
       <ignition_frame_id>lidar_link</ignition_frame_id>
-      <topic>/scan</topic>
+      <topic>scan</topic>
       <update_rate>10</update_rate>
       <ray>
@@ -341,4 +341,100 @@
     <origin xyz="0.099 0 -0.0043" rpy="0 0 0"/>
   </joint>
+  <!-- ============================================= -->
+  <!-- IMU - Inertial Measurement Unit              -->
+  <!-- ============================================= -->
+  <link name="imu_link">
+    <inertial>
+      <origin xyz="0 0 0" rpy="0 0 0"/>
+      <mass value="0.01"/>
+      <inertia ixx="1e-6" ixy="0" ixz="0" iyy="1e-6" iyz="0" izz="1e-6"/>
+    </inertial>
+    <visual>
+      <origin xyz="0 0 0" rpy="0 0 0"/>
+      <geometry>
+        <box size="0.02 0.02 0.02"/>
+      </geometry>
+      <material name="DarkBlue">
+        <color rgba="0.5 0.5 0.5 1"/>
+      </material>
+    </visual>
+    <collision>
+      <origin xyz="0 0 0" rpy="0 0 0"/>
+      <geometry>
+        <box size="0.02 0.02 0.02"/>
+      </geometry>
+    </collision>
+  </link>
+  <joint name="imu_joint" type="fixed">
+    <parent link="chassis_link"/>
+    <child link="imu_link"/>
+    <!-- Positioned at the CoM of the chassis_link -->
+    <origin xyz="0.0099132 0.00030561 0.03955" rpy="0 0 0"/>
+  </joint>
+  <gazebo reference="imu_link">
+    <sensor name="imu_sensor" type="imu">
+      <ignition_frame_id>imu_link</ignition_frame_id>
+      <plugin filename="ignition-gazebo-imu-system" name="ignition::gazebo::systems::Imu">
+      </plugin>
+      <topic>imu</topic>
+      <always_on>true</always_on>
+      <update_rate>100</update_rate>
+      <visualize>true</visualize>
+      <imu>
+        <angular_velocity>
+          <x>
+            <noise type="gaussian">
+              <mean>0.0</mean>
+              <stddev>2e-4</stddev>
+              <bias_mean>0.0000075</bias_mean>
+              <bias_stddev>0.0000008</bias_stddev>
+            </noise>
+          </x>
+          <y>
+            <noise type="gaussian">
+              <mean>0.0</mean>
+              <stddev>2e-4</stddev>
+              <bias_mean>0.0000075</bias_mean>
+              <bias_stddev>0.0000008</bias_stddev>
+            </noise>
+          </y>
+          <z>
+            <noise type="gaussian">
+              <mean>0.0</mean>
+              <stddev>2e-4</stddev>
+              <bias_mean>0.0000075</bias_mean>
+              <bias_stddev>0.0000008</bias_stddev>
+            </noise>
+          </z>
+        </angular_velocity>
+        <linear_acceleration>
+          <x>
+            <noise type="gaussian">
+              <mean>0.0</mean>
+              <stddev>1.7e-2</stddev>
+              <bias_mean>0.1</bias_mean>
+              <bias_stddev>0.001</bias_stddev>
+            </noise>
+          </x>
+          <y>
+            <noise type="gaussian">
+              <mean>0.0</mean>
+              <stddev>1.7e-2</stddev>
+              <bias_mean>0.1</bias_mean>
+              <bias_stddev>0.001</bias_stddev>
+            </noise>
+          </y>
+          <z>
+            <noise type="gaussian">
+              <mean>0.0</mean>
+              <stddev>1.7e-2</stddev>
+              <bias_mean>0.1</bias_mean>
+              <bias_stddev>0.001</bias_stddev>
+            </noise>
+          </z>
+        </linear_acceleration>
+      </imu>
+    </sensor>
+  </gazebo>
   <ros2_control name="IgnitionSystem" type="system">
     <hardware>

Commit message: Updated launch files and added SLAM configuration

File: urdf/assem_urdf.urdf.xacro (robot description, xacro)
@@ -229,10 +229,10 @@
         value="0.1" />
       <inertia
-        ixx="0"
+        ixx="0.0001"
         ixy="0"
         ixz="0"
-        iyy="0"
+        iyy="0.0001"
         iyz="0"
-        izz="0" />
+        izz="0.0001" />
     </inertial>
     <visual>
@@ -336,4 +336,86 @@
     </collision>
   </link>
+  <link name="imu_link">
+    <visual>
+      <geometry>
+        <box size="0.001 0.001 0.001"/>
+      </geometry>
+    </visual>
+    <collision>
+      <geometry>
+        <box size="0.001 0.001 0.001"/>
+      </geometry>
+    </collision>
+  </link>
+  <gazebo reference="imu_link">
+    <sensor name="imu_sensor" type="imu">
+      <ignition_frame_id>imu_link</ignition_frame_id>
+      <plugin filename="ignition-gazebo-imu-system" name="ignition::gazebo::systems::Imu">
+        <topic>/imu</topic>
+      </plugin>
+      <always_on>true</always_on>
+      <update_rate>100</update_rate>
+      <visualize>true</visualize>
+      <imu>
+        <angular_velocity>
+          <x>
+            <noise type="gaussian">
+              <mean>0.0</mean>
+              <stddev>2e-4</stddev>
+              <bias_mean>0.0000075</bias_mean>
+              <bias_stddev>0.0000008</bias_stddev>
+            </noise>
+          </x>
+          <y>
+            <noise type="gaussian">
+              <mean>0.0</mean>
+              <stddev>2e-4</stddev>
+              <bias_mean>0.0000075</bias_mean>
+              <bias_stddev>0.0000008</bias_stddev>
+            </noise>
+          </y>
+          <z>
+            <noise type="gaussian">
+              <mean>0.0</mean>
+              <stddev>2e-4</stddev>
+              <bias_mean>0.0000075</bias_mean>
+              <bias_stddev>0.0000008</bias_stddev>
+            </noise>
+          </z>
+        </angular_velocity>
+        <linear_acceleration>
+          <x>
+            <noise type="gaussian">
+              <mean>0.0</mean>
+              <stddev>1.7e-2</stddev>
+              <bias_mean>0.1</bias_mean>
+              <bias_stddev>0.001</bias_stddev>
+            </noise>
+          </x>
+          <y>
+            <noise type="gaussian">
+              <mean>0.0</mean>
+              <stddev>1.7e-2</stddev>
+              <bias_mean>0.1</bias_mean>
+              <bias_stddev>0.001</bias_stddev>
+            </noise>
+          </y>
+          <z>
+            <noise type="gaussian">
+              <mean>0.0</mean>
+              <stddev>1.7e-2</stddev>
+              <bias_mean>0.1</bias_mean>
+              <bias_stddev>0.001</bias_stddev>
+            </noise>
+          </z>
+        </linear_acceleration>
+      </imu>
+    </sensor>
+  </gazebo>
+  <joint name="imu_joint" type="fixed">
+    <parent link="chassis_link"/>
+    <child link="imu_link"/>
+    <origin xyz="0 0 0.01"/>
+  </joint>
   <joint name="caster_joint" type="fixed">
     <parent link="chassis_link"/>
@@ -394,5 +476,5 @@
         </clip>
       </camera>
-      <cameraName>depth_camera</cameraName>
+z      <cameraName>depth_camera</cameraName>
       <alwaysOn>true</alwaysOn>
       <updateRate>10</updateRate>

Commit message: Sửa lỗi trong urdf và cấu hình SLAM Toolbox, xóa file completion.launch.py

File: urdf/assem_urdf.urdf.xacro (robot description, xacro)
@@ -423,100 +423,4 @@
     <origin xyz="0.099 0 -0.0043" rpy="0 0 0"/>
   </joint>
-  <!-- ============================================= -->
-  <!-- IMU - Inertial Measurement Unit              -->
-  <!-- ============================================= -->
-  <link name="imu_link">
-    <inertial>
-      <origin xyz="0 0 0" rpy="0 0 0"/>
-      <mass value="0.01"/>
-      <inertia ixx="1e-6" ixy="0" ixz="0" iyy="1e-6" iyz="0" izz="1e-6"/>
-    </inertial>
-    <visual>
-      <origin xyz="0 0 0" rpy="0 0 0"/>
-      <geometry>
-        <box size="0.02 0.02 0.02"/>
-      </geometry>
-      <material name="DarkBlue">
-        <color rgba="0.5 0.5 0.5 1"/>
-      </material>
-    </visual>
-    <collision>
-      <origin xyz="0 0 0" rpy="0 0 0"/>
-      <geometry>
-        <box size="0.02 0.02 0.02"/>
-      </geometry>
-    </collision>
-  </link>
-  <joint name="imu_joint" type="fixed">
-    <parent link="chassis_link"/>
-    <child link="imu_link"/>
-    <!-- Positioned at the CoM of the chassis_link -->
-    <origin xyz="0.0099132 0.00030561 0.03955" rpy="0 0 0"/>
-  </joint>
-  <gazebo reference="imu_link">
-    <sensor name="imu_sensor" type="imu">
-      <ignition_frame_id>imu_link</ignition_frame_id>
-      <plugin filename="ignition-gazebo-imu-system" name="ignition::gazebo::systems::Imu">
-      </plugin>
-      <topic>imu</topic>
-      <always_on>true</always_on>
-      <update_rate>100</update_rate>
-      <visualize>true</visualize>
-      <imu>
-        <angular_velocity>
-          <x>
-            <noise type="gaussian">
-              <mean>0.0</mean>
-              <stddev>2e-4</stddev>
-              <bias_mean>0.0000075</bias_mean>
-              <bias_stddev>0.0000008</bias_stddev>
-            </noise>
-          </x>
-          <y>
-            <noise type="gaussian">
-              <mean>0.0</mean>
-              <stddev>2e-4</stddev>
-              <bias_mean>0.0000075</bias_mean>
-              <bias_stddev>0.0000008</bias_stddev>
-            </noise>
-          </y>
-          <z>
-            <noise type="gaussian">
-              <mean>0.0</mean>
-              <stddev>2e-4</stddev>
-              <bias_mean>0.0000075</bias_mean>
-              <bias_stddev>0.0000008</bias_stddev>
-            </noise>
-          </z>
-        </angular_velocity>
-        <linear_acceleration>
-          <x>
-            <noise type="gaussian">
-              <mean>0.0</mean>
-              <stddev>1.7e-2</stddev>
-              <bias_mean>0.1</bias_mean>
-              <bias_stddev>0.001</bias_stddev>
-            </noise>
-          </x>
-          <y>
-            <noise type="gaussian">
-              <mean>0.0</mean>
-              <stddev>1.7e-2</stddev>
-              <bias_mean>0.1</bias_mean>
-              <bias_stddev>0.001</bias_stddev>
-            </noise>
-          </y>
-          <z>
-            <noise type="gaussian">
-              <mean>0.0</mean>
-              <stddev>1.7e-2</stddev>
-              <bias_mean>0.1</bias_mean>
-              <bias_stddev>0.001</bias_stddev>
-            </noise>
-          </z>
-        </linear_acceleration>
-      </imu>
-    </sensor>
-  </gazebo>
   <ros2_control name="IgnitionSystem" type="system">
     <hardware>
@@ -572,5 +476,5 @@
         </clip>
       </camera>
-z      <cameraName>depth_camera</cameraName>
+      <cameraName>depth_camera</cameraName>
       <alwaysOn>true</alwaysOn>
       <updateRate>10</updateRate>
